File: pcb/lora-gateway.kicad_pcb (KiCad board)
At the start: 2 copper layers, 0 parts

Commit message: add board + usr es1 connector
Parts:
- added J1: USB_B_Micro, Connector_USB:USB_Micro-B_Amphenol_10103594-0001LF_Horizontal, F.Cu at (41.4, 71.0)
- added J2: Conn_01x06, Connector_PinHeader_2.54mm:PinHeader_1x06_P2.54mm_Vertical, F.Cu at (40.6, 61.0)
- added J3: Conn_01x06, Connector_PinHeader_2.54mm:PinHeader_1x06_P2.54mm_Vertical, F.Cu at (53.3, 81.3)
- added J4: Conn_Coaxial, Connector_Coaxial:SMA_Molex_73251-2120_EdgeMount_Horizontal, F.Cu at (107.0, 77.0)
- added U1: RFM95W-868S2, RF_Module:HOPERF_RFM9XW_SMD, F.Cu at (92.5, 70.0)
- added U2: ATmega2560-16A, Package_QFP:TQFP-100_14x14mm_P0.5mm, F.Cu at (69.8, 71.0)
Other:
- board outline added: 70.8 x 25.8 mm
